Commit message: feat: pushed ros2 version

File: ergodic_sketching_ros/descriptions/iiwa_drawing.urdf.xacro (robot description, xacro)
@@ -5,14 +5,10 @@
 SPDX-License-Identifier: GPL-3.0-only
 -->
-<robot name="iiwa7" xmlns:xacro="http://www.ros.org/wiki/xacro">
+<robot name="iiwa" xmlns:xacro="http://www.ros.org/wiki/xacro">
   <material name="grey">
     <color rgba="0.85 0.85 0.85 0.5"/>
   </material>
-  <!-- Import Rviz colors -->
-  <xacro:include filename="$(find iiwa_description)/urdf/materials.xacro" />
   <!--Import the lbr iiwa macro -->
-  <xacro:include filename="$(find iiwa_description)/urdf/iiwa7.xacro"/>
-  <xacro:arg name="hardware_interface" default="PositionJointInterface"/>
-  <xacro:arg name="robot_name" default="iiwa"/>
+  <xacro:include filename="$(find iiwa_description)/urdf/iiwa.urdf.xacro"/>
   <xacro:arg name="origin_xyz" default="0 0 0"/>
   <xacro:arg name="origin_rpy" default="0 0 0"/>
@@ -20,12 +16,12 @@
   <link name="world"/>
   <!--iiwa-->
-  <xacro:iiwa7 hardware_interface="$(arg hardware_interface)" robot_name="$(arg robot_name)" parent="world">
+  <xacro:iiwa prefix="iiwa_" parent="world">
     <origin xyz="$(arg origin_xyz)" rpy="$(arg origin_rpy)" />
-  </xacro:iiwa7>
+  </xacro:iiwa>
   <link name="pen_link">
   </link>
   <joint name="pen_joint" type="fixed">
     <origin rpy="0 1.5708 0" xyz="0.15 0 0.12"/>
-    <parent link="iiwa_link_ee"/>
+    <parent link="iiwa_tool0"/>
     <child link="pen_link"/>
   </joint>
